File: TinySmps.sch (EAGLE design)
At the start: 30 parts, among them IC1 LM2596S, IC2 TINY85P, J2 POWER_JACK

Commit message: omar changes
Parts:
- removed C13, C14, C7, C8: 100u, resistor:CPOL-EUC
- removed C15: (no value), resistor:CPOL-EUE7.5-16
- removed C16: (no value), resistor:CPOL-USE5-13
- added POWER: (no value), led:LEDSML0805
- added R3: (no value), resistor:R-EU_R1206
- C1: value 100u -> (none); device resistor:CPOL-EUC -> resistor:CPOL-EUE7.5-16
- C2: value 100u -> (none); device resistor:CPOL-EUC -> resistor:CPOL-EUE5-10.5
- C3, C4, C5, C6: value 100u -> (none); device resistor:CPOL-EUC -> rcl:C-EUC1206
Connections:
- new net IN: C1.+, C3.1, C4.1, IC1.VIN, S1.S
- net GND: now also C3.2, C4.2, C5.2, C6.2, R3.1; no longer C13.-, C14.-, C3.-, C4.-, C5.-, C6.-, C7.-, C8.-
- net N$1: now also POWER.C, R3.2; no longer C1.+, C14.+, C2.+, C3.+, C4.+, C5.+, IC1.VIN, S1.S
- net VCC: now also C2.+, C5.1, C6.1, POWER.A; no longer C13.+, C6.+, C7.+, C8.+
Other:
- moved on the sheet: C1, C12, C2, D1, IC1, L1, R1, TRIM, VOUT
